Commit message: feat: use stolen mesh for mobile base

File: my_robot_description/urdf/mobile_base.xacro (robot description, xacro)
@@ -11,6 +11,10 @@
     <link name="base_link">
         <visual>
+            <!-- <geometry>
+                <box size="${base_length} ${base_width} ${base_height}" />
+            </geometry> -->
             <geometry>
-                <box size="${base_length} ${base_width} ${base_height}" />
+                <mesh filename="package://my_robot_description/meshes/waffle_base.stl"
+                    scale="0.002 0.002 0.002" />
             </geometry>
             <origin xyz="0 0 ${base_height/2}" rpy="0 0 0" />

Commit message: feat: add collision to everything

File: my_robot_description/urdf/mobile_base.xacro (robot description, xacro)
@@ -21,4 +21,10 @@
             <material name="blue" />
         </visual>
+        <collision>
+            <geometry>
+                <box size="${base_length} ${base_width} ${base_height}" />
+            </geometry>
+            <origin xyz="0 0 ${base_height/2}" rpy="0 0 0" />
+        </collision>
         <xacro:box_inertia
             m="5.0" x="${base_length}" y="${base_width}" z="${base_height}"
@@ -35,4 +41,10 @@
                 <material name="grey" />
             </visual>
+            <collision>
+                <geometry>
+                    <sphere radius="${wheel_radius}" />
+                </geometry>
+                <origin xyz="0 0 0" rpy="${pi/2} 0 0" />
+            </collision>
             <xacro:solid_cylinder_inertia
                 m="1.0" r="${wheel_radius}" l="${wheel_length}"
@@ -51,4 +63,10 @@
             <material name="grey" />
         </visual>
+        <collision>
+            <geometry>
+                <sphere radius="${caster_wheel_radius}" />
+            </geometry>
+            <origin xyz="0 0 0" rpy="0 0 0" />
+        </collision>
         <xacro:solid_sphere_inertia
             m="0.5" r="${caster_wheel_radius}"
