Commit message: feat: add inertia for the box

File: my_robot_description/urdf/common_properties.xacro (robot description, xacro)
@@ -7,3 +7,14 @@
         <color rgba="0.5 0.5 0.5 1" />
     </material>
+    <xacro:macro name="box_inertia" params="m x y z o_xyz o_rpy">
+        <inertial>
+            <mass value="${m}" />
+            <origin xyz="${o_xyz}" rpy="${o_rpy}" />
+            <inertia
+                ixx="${(m/12) * (y*y + z*z)}" ixy="0" ixz="0"
+                iyy="${(m/12) * (x*x + z*z)}" iyz="0"
+                izz="${(m/12) * (x*x + y*y)}"
+            />
+        </inertial>
+    </xacro:macro>
 </robot>

File: my_robot_description/urdf/mobile_base.xacro (robot description, xacro)
@@ -11,14 +11,18 @@
     <link name="base_link">
         <visual>
+            <geometry>
+                <box size="${base_length} ${base_width} ${base_height}" />
+            </geometry>
             <!-- <geometry>
-                <box size="${base_length} ${base_width} ${base_height}" />
-            </geometry> -->
-            <geometry>
                 <mesh filename="package://my_robot_description/meshes/waffle_base.stl"
                     scale="0.002 0.002 0.002" />
-            </geometry>
+            </geometry> -->
             <origin xyz="0 0 ${base_height/2}" rpy="0 0 0" />
             <material name="blue" />
         </visual>
+        <xacro:box_inertia
+            m="5.0" x="${base_length}" y="${base_width}" z="${base_height}"
+            o_xyz="0 0 ${base_height/2}" o_rpy="0 0 0"
+        />
     </link>
     <xacro:macro name="wheel_link" params="prefix">

Commit message: feat: add inertia for all wheels

File: my_robot_description/urdf/common_properties.xacro (robot description, xacro)
@@ -18,3 +18,25 @@
         </inertial>
     </xacro:macro>
+    <xacro:macro name="solid_sphere_inertia" params="m r o_xyz o_rpy">
+        <inertial>
+            <mass value="${m}" />
+            <origin xyz="${o_xyz}" rpy="${o_rpy}" />
+            <inertia
+                ixx="${(2/5)*m*r*r}" ixy="0" ixz="0"
+                iyy="${(2/5)*m*r*r}" iyz="0"
+                izz="${(2/5)*m*r*r}"
+            />
+        </inertial>
+    </xacro:macro>
+    <xacro:macro name="solid_cylinder_inertia" params="m r l o_xyz o_rpy">
+        <inertial>
+            <mass value="${m}" />
+            <origin xyz="${o_xyz}" rpy="${o_rpy}" />
+            <inertia
+                ixx="${(m/12)*(3*r*r + l*l)}" ixy="0" ixz="0"
+                iyy="${(m/12)*(3*r*r + l*l)}" iyz="0"
+                izz="${(m/2)*(r*r)}"
+            />
+        </inertial>
+    </xacro:macro>
 </robot>

File: my_robot_description/urdf/mobile_base.xacro (robot description, xacro)
@@ -35,4 +35,8 @@
                 <material name="grey" />
             </visual>
+            <xacro:solid_cylinder_inertia
+                m="1.0" r="${wheel_radius}" l="${wheel_length}"
+                o_xyz="0 0 0" o_rpy="${pi/2} 0 0"
+            />
         </link>
     </xacro:macro>
@@ -47,4 +51,8 @@
             <material name="grey" />
         </visual>
+        <xacro:solid_sphere_inertia
+            m="0.5" r="${caster_wheel_radius}"
+            o_xyz="0 0 0" o_rpy="0 0 0"
+        />
     </link>
     <joint name="base_joint" type="fixed">

Commit message: feat: add a base for the arm on top of the robot

File: my_robot_description/urdf/common_properties.xacro (robot description, xacro)
@@ -6,4 +6,7 @@
     <material name="grey">
         <color rgba="0.5 0.5 0.5 1" />
+    </material>
+    <material name="orange">
+        <color rgba="1.0 0.5 0.0 1" />
     </material>
     <xacro:macro name="box_inertia" params="m x y z o_xyz o_rpy">

File: my_robot_description/urdf/my_robot.urdf.xacro (robot description, xacro)
@@ -5,3 +5,4 @@
     <xacro:include filename="mobile_base_gazebo.xacro" />
     <xacro:include filename="camera.xacro" />
+    <xacro:include filename="arm.xacro" />
 </robot>
