Commit message: feat: collision and inertia for arm base

File: my_robot_description/urdf/arm.xacro (robot description, xacro)
@@ -4,12 +4,23 @@
     <xacro:property name="arm_base_width" value="0.1" />
     <xacro:property name="arm_base_height" value="0.02" />
+    <xacro:property name="arm_segment_length" value="0.3" />
+    <xacro:property name="arm_segment_radius" value="0.02" />
     <link name="arm_base_link">
         <visual>
             <geometry>
-                <box size="0.1 0.1 0.02" />
+                <box size="${arm_base_length} ${arm_base_width} ${arm_base_height}" />
             </geometry>
             <material name="orange" />
             <origin xyz="0 0 0" rpy="0 0 0" />
         </visual>
+        <collision>
+            <geometry>
+                <box size="${arm_base_length} ${arm_base_width} ${arm_base_height}" />
+            </geometry>
+        </collision>
+        <xacro:box_inertia
+            m="0.5" x="${arm_base_length}" y="${arm_base_width}" z="${arm_base_height}"
+            o_xyz="0 0 0" o_rpy="0 0 0"
+        />
     </link>
     <!-- <link name="forearm_link"></link>

Commit message: feat: first segment of arm

File: my_robot_description/urdf/arm.xacro (robot description, xacro)
@@ -24,6 +24,23 @@
         />
     </link>
-    <!-- <link name="forearm_link"></link>
-    <link name="hand_link"></link> -->
+    <link name="forearm_link">
+        <visual>
+            <geometry>
+                <cylinder radius="${arm_segment_radius}" length="${arm_segment_length}" />
+            </geometry>
+            <material name="yellow" />
+            <origin xyz="0 0 0" rpy="0 0 0" />
+        </visual>
+        <collision>
+            <geometry>
+                <cylinder radius="${arm_segment_radius}" length="${arm_segment_length}" />
+            </geometry>
+        </collision>
+        <xacro:solid_cylinder_inertia
+            m="0.3" r="${arm_segment_radius}" l="${arm_segment_length}"
+            o_xyz="0 0 0" o_rpy="0 0 0"
+        />
+    </link>
+    <!-- <link name="hand_link"></link> -->
     <joint name="base_arm_base_joint" type="fixed">
         <parent link="base_link" />
@@ -31,3 +48,8 @@
         <origin xyz="0 0 ${base_height + arm_base_height/2}" rpy="0 0 0" />
     </joint>
+    <joint name="arm_base_forearm_joint" type="fixed">
+        <parent link="arm_base_link" />
+        <child link="forearm_link" />
+        <origin xyz="0 0 ${arm_segment_length/2 + arm_base_height/2}" rpy="0 0 0" />
+    </joint>
 </robot>

File: my_robot_description/urdf/common_properties.xacro (robot description, xacro)
@@ -9,4 +9,7 @@
     <material name="orange">
         <color rgba="1.0 0.5 0.0 1" />
+    </material>
+    <material name="yellow">
+        <color rgba="1.0 1.0 0.0 1" />
     </material>
     <xacro:macro name="box_inertia" params="m x y z o_xyz o_rpy">

Commit message: feat: add second segment of arm

File: my_robot_description/urdf/arm.xacro (robot description, xacro)
@@ -42,5 +42,22 @@
         />
     </link>
-    <!-- <link name="hand_link"></link> -->
+    <link name="hand_link">
+        <visual>
+            <geometry>
+                <cylinder radius="${arm_segment_radius}" length="${arm_segment_length}" />
+            </geometry>
+            <material name="grey" />
+            <origin xyz="0 0 0" rpy="0 0 0" />
+        </visual>
+        <collision>
+            <geometry>
+                <cylinder radius="${arm_segment_radius}" length="${arm_segment_length}" />
+            </geometry>
+        </collision>
+        <xacro:solid_cylinder_inertia
+            m="0.3" r="${arm_segment_radius}" l="${arm_segment_length}"
+            o_xyz="0 0 0" o_rpy="0 0 0"
+        />
+    </link>
     <joint name="base_arm_base_joint" type="fixed">
         <parent link="base_link" />
@@ -53,3 +70,8 @@
         <origin xyz="0 0 ${arm_segment_length/2 + arm_base_height/2}" rpy="0 0 0" />
     </joint>
+    <joint name="forearm_hand_joint" type="fixed">
+        <parent link="forearm_link" />
+        <child link="hand_link" />
+        <origin xyz="0 0 ${arm_segment_length}" rpy="0 0 0" />
+    </joint>
 </robot>

Commit message: feat: make arm segments movable by making sure joints are correctly placed
Also: move arm base forward slightly so it can move freely.

File: my_robot_description/urdf/arm.xacro (robot description, xacro)
@@ -30,5 +30,5 @@
             </geometry>
             <material name="yellow" />
-            <origin xyz="0 0 0" rpy="0 0 0" />
+            <origin xyz="0 0 ${arm_segment_length/2}" rpy="0 0 0" />
         </visual>
         <collision>
@@ -47,6 +47,6 @@
                 <cylinder radius="${arm_segment_radius}" length="${arm_segment_length}" />
             </geometry>
-            <material name="grey" />
-            <origin xyz="0 0 0" rpy="0 0 0" />
+            <material name="yellow" />
+            <origin xyz="0 0 ${arm_segment_length/2}" rpy="0 0 0" />
         </visual>
         <collision>
@@ -63,15 +63,19 @@
         <parent link="base_link" />
         <child link="arm_base_link" />
-        <origin xyz="0 0 ${base_height + arm_base_height/2}" rpy="0 0 0" />
+        <origin xyz="${base_length/4} 0 ${base_height + arm_base_height/2}" rpy="0 0 0" />
     </joint>
-    <joint name="arm_base_forearm_joint" type="fixed">
+    <joint name="arm_base_forearm_joint" type="revolute">
         <parent link="arm_base_link" />
         <child link="forearm_link" />
-        <origin xyz="0 0 ${arm_segment_length/2 + arm_base_height/2}" rpy="0 0 0" />
+        <origin xyz="0 0 ${arm_base_height/2}" rpy="0 0 0" />
+        <axis xyz="0 1 0" />
+        <limit lower="0" upper="${pi/2}" effort="10" velocity="10" />
     </joint>
-    <joint name="forearm_hand_joint" type="fixed">
+    <joint name="forearm_hand_joint" type="revolute">
         <parent link="forearm_link" />
         <child link="hand_link" />
         <origin xyz="0 0 ${arm_segment_length}" rpy="0 0 0" />
+        <axis xyz="0 1 0" />
+        <limit lower="0" upper="${pi/2}" effort="10" velocity="10" />
     </joint>
 </robot>

Commit message: fix: use limits and dynamics values from pdf spec

File: my_robot_description/urdf/arm.xacro (robot description, xacro)
@@ -70,5 +70,6 @@
         <origin xyz="0 0 ${arm_base_height/2}" rpy="0 0 0" />
         <axis xyz="0 1 0" />
-        <limit lower="0" upper="${pi/2}" effort="10" velocity="10" />
+        <limit lower="0" upper="${pi/2}" effort="100" velocity="100" />
+        <dynamics friction="0.3" damping="0.3" />
     </joint>
     <joint name="forearm_hand_joint" type="revolute">
@@ -77,5 +78,6 @@
         <origin xyz="0 0 ${arm_segment_length}" rpy="0 0 0" />
         <axis xyz="0 1 0" />
-        <limit lower="0" upper="${pi/2}" effort="10" velocity="10" />
+        <limit lower="0" upper="${pi/2}" effort="100" velocity="100" />
+        <dynamics friction="0.3" damping="0.3" />
     </joint>
 </robot>

Commit message: fix: make sure joints are properly placed

File: my_robot_description/urdf/arm.xacro (robot description, xacro)
@@ -12,5 +12,5 @@
             </geometry>
             <material name="orange" />
-            <origin xyz="0 0 0" rpy="0 0 0" />
+            <origin xyz="0 0 ${arm_base_height/2}" rpy="0 0 0" />
         </visual>
         <collision>
@@ -21,5 +21,5 @@
         <xacro:box_inertia
             m="0.5" x="${arm_base_length}" y="${arm_base_width}" z="${arm_base_height}"
-            o_xyz="0 0 0" o_rpy="0 0 0"
+            o_xyz="0 0 ${arm_base_height/2}" o_rpy="0 0 0"
         />
     </link>
@@ -63,10 +63,10 @@
         <parent link="base_link" />
         <child link="arm_base_link" />
-        <origin xyz="${base_length/4} 0 ${base_height + arm_base_height/2}" rpy="0 0 0" />
+        <origin xyz="${base_length/4} 0 ${base_height}" rpy="0 0 0" />
     </joint>
     <joint name="arm_base_forearm_joint" type="revolute">
         <parent link="arm_base_link" />
         <child link="forearm_link" />
-        <origin xyz="0 0 ${arm_base_height/2}" rpy="0 0 0" />
+        <origin xyz="0 0 ${arm_base_height}" rpy="0 0 0" />
         <axis xyz="0 1 0" />
         <limit lower="0" upper="${pi/2}" effort="100" velocity="100" />

Commit message: fix: collision should have origin too

File: my_robot_description/urdf/arm.xacro (robot description, xacro)
@@ -18,4 +18,5 @@
                 <box size="${arm_base_length} ${arm_base_width} ${arm_base_height}" />
             </geometry>
+            <origin xyz="0 0 ${arm_base_height/2}" rpy="0 0 0" />
         </collision>
         <xacro:box_inertia

Commit message: fix: make sure collision and inerta have the same origins as the visuals

File: my_robot_description/urdf/arm.xacro (robot description, xacro)
@@ -37,8 +37,9 @@
                 <cylinder radius="${arm_segment_radius}" length="${arm_segment_length}" />
             </geometry>
+            <origin xyz="0 0 ${arm_segment_length/2}" rpy="0 0 0" />
         </collision>
         <xacro:solid_cylinder_inertia
             m="0.3" r="${arm_segment_radius}" l="${arm_segment_length}"
-            o_xyz="0 0 0" o_rpy="0 0 0"
+            o_xyz="0 0 ${arm_segment_length/2}" o_rpy="0 0 0"
         />
     </link>
@@ -55,8 +56,9 @@
                 <cylinder radius="${arm_segment_radius}" length="${arm_segment_length}" />
             </geometry>
+            <origin xyz="0 0 ${arm_segment_length/2}" rpy="0 0 0" />
         </collision>
         <xacro:solid_cylinder_inertia
             m="0.3" r="${arm_segment_radius}" l="${arm_segment_length}"
-            o_xyz="0 0 0" o_rpy="0 0 0"
+            o_xyz="0 0 ${arm_segment_length/2}" o_rpy="0 0 0"
         />
     </link>
